File: USB-to-UART-Bridge.kicad_sch (KiCad schematic)
At the start: 30 parts, among them J1 USB_C_Receptacle_USB2.0, J2 Conn_02x10_Odd_Even, J3 Conn_01x06, J4 Conn_01x06, Q1 BC848, Q2 BC848, U1 USBLC6-2SC6, U2 CP2102N-Axx-xQFN24, U3 MCP1703A-3302_SOT223

Commit message: Updated BOM
Parts:
- C1, C3: MPN (none) -> CL10A475KO8NNNC
- C2, C4: MPN (none) -> C0603C104K5RACTU
- C5, C6: MPN (none) -> CC0603KRX7R7BB105
- D1, D2: MPN (none) -> LTST-C190KRKT
- D3: MPN (none) -> LTST-C190KGKT
- F1: MPN (none) -> PTSA120613V050
- J1: MPN (none) -> DX07S016JA3R1500
- J2: MPN (none) -> 087-2-020-0-S-XS0-1260
- J3, J4: MPN (none) -> B6B-XH-A(LF)(SN)
- Q1, Q2: MPN (none) -> BC848BLT3G
- R1, R2: value 5.1k -> 5k1; MPN (none) -> Res 0603 5k1 1%
- R10, R11, R7: MPN (none) -> Res 0603 10k 1%
- R3, R6, R8, R9: MPN (none) -> Res 0603 1k 1%
- R4: value 22.1k -> 22k1; MPN (none) -> Res 0603 22k1 1%
- R5: value 47.5k -> 47k5; MPN (none) -> Res 0603 47k5 1%
- U1: MPN (none) -> USBLC6-2SC6
- U2: MPN (none) -> CP2102N-A02-GQFN24R
- U3: MPN (none) -> MCP1703-3302E/DB
Changed lines of the file:
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@@
+      (effects (font (size 1.27 1.27)) hide)
+    )
+    (property "MPN" "Res 0603 1k 1%" (id 4) (at 180.34 48.26 0)
       (effects (font (size 1.27 1.27)) hide)
     )
@@
     )
     (property "Datasheet" "~" (id 3) (at 109.22 43.18 0)
+      (effects (font (size 1.27 1.27)) hide)
+    )
+    (property "MPN" "CC0603KRX7R7BB105" (id 4) (at 109.22 43.18 0)
       (effects (font (size 1.27 1.27)) hide)
     )
@@
       (effects (font (size 1.27 1.27)) hide)
     )
+    (property "MPN" "CC0603KRX7R7BB105" (id 4) (at 133.35 43.18 0)
+      (effects (font (size 1.27 1.27)) hide)
+    )
     (pin "1")
     (pin "2")
@@
       (effects (font (size 1.27 1.27)) hide)
     )
+    (property "MPN" "LTST-C190KRKT" (id 4) (at 82.55 44.45 0)
+      (effects (font (size 1.27 1.27)) hide)
+    )
     (pin "1")
     (pin "2")
@@
       (effects (font (size 1.27 1.27)) hide)
     )
+    (property "MPN" "Res 0603 1k 1%" (id 5) (at 251.46 83.82 0)
+      (effects (font (size 1.27 1.27)) hide)
+    )
     (pin "1")
     (pin "2")
@@
     )
     (property "Datasheet" "~" (id 3) (at 271.78 147.32 0)
+      (effects (font (size 1.27 1.27)) hide)
+    )
+    (property "MPN" "B6B-XH-A(LF)(SN)" (id 4) (at 271.78 147.32 0)
       (effects (font (size 1.27 1.27)) hide)
     )
@@
       (effects (font (size 1.27 1.27)) hide)
     )
+    (property "MPN" "USBLC6-2SC6" (id 5) (at 121.92 71.12 0)
+      (effects (font (size 1.27 1.27)) hide)
+    )
     (pin "1")
     (pin "2")
@@
       (effects (font (size 1.27 1.27)) hide)
     )
+    (property "MPN" "Res 0603 10k 1%" (id 4) (at 227.33 78.74 0)
+      (effects (font (size 1.27 1.27)) hide)
+    )
     (pin "1")
     (pin "2")
@@
       (effects (font (size 1.27 1.27)) hide)
     )
+    (property "MPN" "LTST-C190KGKT" (id 4) (at 259.08 88.9 0)
+      (effects (font (size 1.27 1.27)) hide)
+    )
     (pin "1")
     (pin "2")
@@
     (in_bom yes) (on_board yes)
     (property "Reference" "R1" (id 0) (at 67.31 41.91 90))
-    (property "Value" "5.1k" (id 1) (at 58.42 41.91 90))
+    (property "Value" "5k1" (id 1) (at 58.42 41.91 90))
     (property "Footprint" "Resistor_SMD:R_0603_1608Metric" (id 2) (at 63.5 43.18 0)
       (effects (font (size 1.27 1.27)) hide)
@@
     )
     (property "LCSC" "C25905" (id 4) (at 63.5 43.18 0)
+      (effects (font (size 1.27 1.27)) hide)
+    )
+    (property "MPN" "Res 0603 5k1 1%" (id 5) (at 63.5 43.18 0)
       (effects (font (size 1.27 1.27)) hide)
     )
@@
       (effects (font (size 1.27 1.27)) hide)
     )
+    (property "MPN" "PTSA120613V050" (id 4) (at 63.5 38.1 0)
+      (effects (font (size 1.27 1.27)) hide)
+    )
     (pin "1")
     (pin "2")
@@
     )
     (property "Datasheet" "~" (id 3) (at 254 50.8 0)
+      (effects (font (size 1.27 1.27)) hide)
+    )
+    (property "MPN" "087-2-020-0-S-XS0-1260" (id 4) (at 254 50.8 0)
       (effects (font (size 1.27 1.27)) hide)
     )
@@
       (effects (font (size 1.27 1.27)) (justify left) hide)
     )
+    (property "MPN" "BC848BLT3G" (id 4) (at 189.23 132.08 0)
+      (effects (font (size 1.27 1.27)) hide)
+    )
     (pin "1")
     (pin "2")
@@
       (effects (font (size 1.27 1.27)) hide)
     )
+    (property "MPN" "Res 0603 10k 1%" (id 5) (at 177.8 132.08 0)
+      (effects (font (size 1.27 1.27)) hide)
+    )
     (pin "1")
     (pin "2")
@@
       (effects (font (size 1.27 1.27)) (justify left))
     )
-    (property "Value" "22.1k" (id 1) (at 165.1 57.1499 0)
+    (property "Value" "22k1" (id 1) (at 165.1 57.1499 0)
       (effects (font (size 1.27 1.27)) (justify left))
     )
@@
       (effects (font (size 1.27 1.27)) hide)
     )
+    (property "MPN" "Res 0603 22k1 1%" (id 4) (at 162.56 55.88 0)
+      (effects (font (size 1.27 1.27)) hide)
+    )
     (pin "1")
     (pin "2")
@@
     )
     (property "Datasheet" "~" (id 3) (at 251.46 88.9 90)
+      (effects (font (size 1.27 1.27)) hide)
+    )
+    (property "MPN" "LTST-C190KRKT" (id 4) (at 251.46 88.9 0)
       (effects (font (size 1.27 1.27)) hide)
     )
@@
       (effects (font (size 1.27 1.27)) (justify left) hide)
     )
+    (property "MPN" "BC848BLT3G" (id 4) (at 189.23 148.59 0)
+      (effects (font (size 1.27 1.27)) hide)
+    )
     (pin "1")
     (pin "2")
@@
       (effects (font (size 1.27 1.27)) hide)
     )
+    (property "MPN" "Res 0603 1k 1%" (id 5) (at 259.08 83.82 0)
+      (effects (font (size 1.27 1.27)) hide)
+    )
     (pin "1")
     (pin "2")
@@
       (effects (font (size 1.27 1.27)) hide)
     )
+    (property "MPN" "CL10A475KO8NNNC" (id 4) (at 212.09 39.37 0)
+      (effects (font (size 1.27 1.27)) hide)
+    )
     (pin "1")
     (pin "2")
@@
     (in_bom yes) (on_board yes)
     (property "Reference" "R2" (id 0) (at 67.31 44.45 90))
-    (property "Value" "5.1k" (id 1) (at 58.42 44.45 90))
+    (property "Value" "5k1" (id 1) (at 58.42 44.45 90))
     (property "Footprint" "Resistor_SMD:R_0603_1608Metric" (id 2) (at 63.5 45.72 0)
       (effects (font (size 1.27 1.27)) hide)
@@
     )
     (property "LCSC" "C25905" (id 4) (at 63.5 45.72 0)
+      (effects (font (size 1.27 1.27)) hide)
+    )
+    (property "MPN" "Res 0603 5k1 1%" (id 5) (at 63.5 45.72 0)
       (effects (font (size 1.27 1.27)) hide)
     )
@@
       (effects (font (size 1.27 1.27)) (justify right))
     )
-    (property "Value" "47.5k" (id 1) (at 168.91 66.0399 0)
+    (property "Value" "47k5" (id 1) (at 168.91 66.0399 0)
       (effects (font (size 1.27 1.27)) (justify right))
     )
@@
     )
     (property "Datasheet" "~" (id 3) (at 171.45 64.77 0)
+      (effects (font (size 1.27 1.27)) hide)
+    )
+    (property "MPN" "Res 0603 47k5 1%" (id 4) (at 171.45 64.77 0)
       (effects (font (size 1.27 1.27)) hide)
     )
@@
       (effects (font (size 1.27 1.27)) hide)
     )
+    (property "MPN" "MCP1703-3302E/DB" (id 4) (at 121.92 38.1 0)
+      (effects (font (size 1.27 1.27)) hide)
+    )
     (pin "1")
     (pin "2")
@@
       (effects (font (size 1.27 1.27)) hide)
     )
+    (property "MPN" "C0603C104K5RACTU" (id 4) (at 184.15 39.37 0)
+      (effects (font (size 1.27 1.27)) hide)
+    )
     (pin "1")
     (pin "2")
@@
       (effects (font (size 1.27 1.27)) hide)
     )
+    (property "MPN" "Res 0603 1k 1%" (id 5) (at 82.55 39.37 0)
+      (effects (font (size 1.27 1.27)) hide)
+    )
     (pin "1")
     (pin "2")
@@
     )
     (property "Datasheet" "https://www.silabs.com/documents/public/data-sheets/cp2102n-datasheet.pdf" (id 3) (at 200.66 90.17 0)
+      (effects (font (size 1.27 1.27)) hide)
+    )
+    (property "MPN" "CP2102N-A02-GQFN24R" (id 4) (at 199.39 71.12 0)
       (effects (font (size 1.27 1.27)) hide)
     )
@@
       (effects (font (size 1.27 1.27)) hide)
     )
+    (property "MPN" "B6B-XH-A(LF)(SN)" (id 4) (at 271.78 127 0)
+      (effects (font (size 1.27 1.27)) hide)
+    )
     (pin "1")
     (pin "2")
@@
       (effects (font (size 1.27 1.27)) hide)
     )
+    (property "MPN" "Res 0603 10k 1%" (id 5) (at 177.8 148.59 0)
+      (effects (font (size 1.27 1.27)) hide)
+    )
     (pin "1")
     (pin "2")
@@
       (effects (font (size 1.27 1.27)) hide)
     )
+    (property "MPN" "C0603C104K5RACTU" (id 4) (at 222.25 39.37 0)
+      (effects (font (size 1.27 1.27)) hide)
+    )
     (pin "1")
     (pin "2")
@@
     )
     (property "Datasheet" "~" (id 3) (at 173.99 39.37 0)
+      (effects (font (size 1.27 1.27)) hide)
+    )
+    (property "MPN" "CL10A475KO8NNNC" (id 4) (at 173.99 39.37 0)
       (effects (font (size 1.27 1.27)) hide)
     )
@@
     )
     (property "Datasheet" "https://www.usb.org/sites/default/files/documents/usb_type-c.zip" (id 3) (at 44.45 53.34 0)
+      (effects (font (size 1.27 1.27)) hide)
+    )
+    (property "MPN" "DX07S016JA3R1500" (id 4) (at 40.64 53.34 0)
       (effects (font (size 1.27 1.27)) hide)
     )
@@
     )
     (path "/56fc849c-b296-4403-9bb4-03c6bcf87048"
-      (reference "R1") (unit 1) (value "5.1k") (footprint "Resistor_SMD:R_0603_1608Metric")
+      (reference "R1") (unit 1) (value "5k1") (footprint "Resistor_SMD:R_0603_1608Metric")
     )
     (path "/b0299914-5178-40c4-9716-29d440fcbc3d"
-      (reference "R2") (unit 1) (value "5.1k") (footprint "Resistor_SMD:R_0603_1608Metric")
+      (reference "R2") (unit 1) (value "5k1") (footprint "Resistor_SMD:R_0603_1608Metric")
     )
     (path "/cd4b51a4-7cec-4fdf-9914-01b4bab25851"
@@
     )
     (path "/97bf3737-ccff-4581-9b59-ee01090732fb"
-      (reference "R4") (unit 1) (value "22.1k") (footprint "Resistor_SMD:R_0603_1608Metric")
+      (reference "R4") (unit 1) (value "22k1") (footprint "Resistor_SMD:R_0603_1608Metric")
     )
     (path "/b29f51b7-69d4-4d97-a81d-c57880f223e3"
-      (reference "R5") (unit 1) (value "47.5k") (footprint "Resistor_SMD:R_0603_1608Metric")
+      (reference "R5") (unit 1) (value "47k5") (footprint "Resistor_SMD:R_0603_1608Metric")
     )
     (path "/120a8b8d-4a70-4759-b067-b948fdd1c60e"
